Commit message: recovered working sensors, slam working. ready for nav2 or drive base change

File: src/robot_description_pkg/urdf/old_robot_current2.urdf (robot description, URDF)
Before this commit: robot terry, 6 links, 5 joints
Links:
- removed link lidar_left
- link base_link: geometry collision box size=0.3 0.2 0.1; visual box size=0.3 0.2 0.1
- link left_wheel: geometry collision cylinder length=0.03 radius=0.05; visual cylinder length=0.03 radius=0.05
- link right_wheel: geometry collision cylinder length=0.03 radius=0.05; visual cylinder length=0.03 radius=0.05
Joints:
- removed joint lidar_left_joint
- removed joint lidar_right_joint
- added joint laser_joint: type fixed, parent base_link, child laser, origin xyz=0.1 0 0.15 rpy=0 0 0
- joint left_wheel_joint: origin xyz=0 0.066675 0 rpy=0 0 0 -> xyz=0 0.115 0 rpy=0 0 0
- joint right_wheel_joint: origin xyz=0 -0.066675 0 rpy=0 0 0 -> xyz=0 -0.115 0 rpy=0 0 0
- joint ultrasonic_joint: origin xyz=0.0762 0 0.127 rpy=0 0 0 -> xyz=0.15 0 0.08 rpy=0 0 0
