Commit message: working backwards mecanum drive

File: src/robot_description_pkg/urdf/mecanum_small.urdf (robot description, URDF)
Before this commit: robot mecanum_robot, 7 links, 6 joints
Links:
- removed link scan
- added link laser, mass 0.05; collision cylinder length=0.04 radius=0.035; visual cylinder length=0.04 radius=0.035
Joints:
- joint scan_joint: child scan -> laser

Commit message: updates to tf tree with odom and state publishing,base footprint component added for nav2

File: src/robot_description_pkg/urdf/mecanum_small.urdf (robot description, URDF)
Before this commit: robot mecanum_robot, 7 links, 6 joints
Links:
- added link base_footprint
Joints:
- added joint base_footprint_to_base_link: type fixed, parent base_link, child base_footprint, origin xyz=0 0 0 rpy=0 0 0

Commit message: starting cv, nav2 mostly working but needs tuned, starting dynamic object following with commanderAPI

File: src/robot_description_pkg/urdf/mecanum_small.urdf (robot description, URDF)
Before this commit: robot mecanum_robot, 8 links, 7 joints
Joints:
- joint scan_joint: origin xyz=0.1 0 0.15 rpy=0 0 0 -> xyz=0.1 0 0.15 rpy=0 0 1.5708

Commit message: simulation development started

File: src/robot_description_pkg/urdf/mecanum_small.urdf (robot description, URDF)
Before this commit: robot mecanum_robot, 8 links, 7 joints
Joints:
- joint front_left_wheel_joint: limit (none) -> effort=10.0 velocity=40.0
- joint front_right_wheel_joint: limit (none) -> effort=10.0 velocity=40.0
- joint rear_left_wheel_joint: limit (none) -> effort=10.0 velocity=40.0
- joint rear_right_wheel_joint: limit (none) -> effort=10.0 velocity=40.0
